Commit message: multiple goal joint alpha

File: src/ros_deep_sampler/urdf/sampler_model1.urdf (robot description, URDF)
Before this commit: robot slider_robot, 5 links, 4 joints
Links:
- removed link platform_link
- added link slider_link, mass 1.0; collision box size=0.1 0.6 0.1; visual box size=0.1 0.6 0.1
Joints:
- joint drill_joint: limit lower=-0.5 upper=0.1 effort=50 velocity=0.5 -> lower=-0.2 upper=0.2 effort=50 velocity=0.5; parent platform_link -> slider_link
- joint platform_joint: child platform_link -> slider_link; limit lower=-0.3 upper=0.3 effort=50 velocity=0.5 -> lower=-0.2 upper=0.2 effort=50 velocity=0.5; origin xyz=0.06 0 0 rpy=0 0 0 -> xyz=0.06 0 1 rpy=0 0 0
- joint rotor_joint: limit (none) -> lower=0.0 upper=6.2 effort=50 velocity=0.5
- joint world_to_base: origin xyz=0 0 1 rpy=0 0 0 -> xyz=0 0 0 rpy=0 0 0
