Commit message: bridge node for can

File: src/ros_deep_sampler/urdf/sampler_model.urdf (robot description, URDF)
Before this commit: robot slider_robot, 5 links, 4 joints
Joints:
- removed joint slider_joint
- added joint platform_joint: type prismatic, parent base_link, child slider_link, origin xyz=0.06 0 1 rpy=0 0 0, axis 0 0 1, limit lower=-0.2 upper=0.2 effort=50 velocity=0.5

Commit message: multiple joints alpha1

File: src/ros_deep_sampler/urdf/sampler_model.urdf (robot description, URDF)
Before this commit: robot slider_robot, 5 links, 4 joints
Joints:
- joint drill_joint: limit lower=-0.5 upper=0.1 effort=50 velocity=0.5 -> effort=50 velocity=0.5

Commit message: drill movement debug

File: src/ros_deep_sampler/urdf/sampler_model.urdf (robot description, URDF)
Before this commit: robot slider_robot, 5 links, 4 joints
Links:
- removed link rotor_link
Joints:
- removed joint rotor_joint
- joint drill_joint: limit effort=50 velocity=0.5 -> lower=-0.2 upper=0.2 effort=500 velocity=0.5
- joint platform_joint: limit lower=-0.3 upper=0.3 effort=50 velocity=0.5 -> lower=-0.4 upper=0.4 effort=500 velocity=0.5

Commit message: rotation implementation

File: src/ros_deep_sampler/urdf/sampler_model.urdf (robot description, URDF)
Before this commit: robot slider_robot, 4 links, 3 joints
Links:
- added link rotor_link, mass 0.5; collision box size=0.07 0.07 0.02; visual box size=0.07 0.07 0.02
Joints:
- added joint rotor_joint: type continuous, parent drill_link, child rotor_link, origin xyz=0 0 -0.3 rpy=0 0 0, axis 0 0 1, limit effort=500 velocity=0.5
- joint drill_joint: limit lower=-0.2 upper=0.2 effort=500 velocity=0.5 -> lower=-0.5 upper=0.5 effort=500 velocity=0.5
- joint world_to_base: origin xyz=0 0 1 rpy=0 0 0 -> xyz=0 0 2 rpy=0 0 0

Commit message: all joints movement

File: src/ros_deep_sampler/urdf/sampler_model.urdf (robot description, URDF)
Before this commit: robot slider_robot, 5 links, 4 joints
Links:
- link drill_link: mass 1.0 -> 3.0
- link platform_link: mass 1.0 -> 5.0
Joints:
- joint drill_joint: limit lower=-0.5 upper=0.5 effort=500 velocity=0.5 -> lower=-0.5 upper=0.5 effort=5000 velocity=0.5
- joint platform_joint: limit lower=-0.4 upper=0.4 effort=500 velocity=0.5 -> lower=-0.5 upper=0.4 effort=1000 velocity=0.3
- joint rotor_joint: limit effort=500 velocity=0.5 -> effort=500 velocity=5
