Commit message: hardware interface to gazebo pos publisher

File: src/ros_deep_sampler/urdf/sampler_model.urdf (robot description, URDF)
Before this commit: robot slider_robot, 5 links, 4 joints
Joints:
- joint platform_joint: limit lower=-0.5 upper=0.4 effort=1000 velocity=0.3 -> lower=-0.5 upper=0.5 effort=5000 velocity=0.5

Commit message: calibration logic plus velocity control for calibration

File: src/ros_deep_sampler/urdf/sampler_model.urdf (robot description, URDF)
Before this commit: robot slider_robot, 5 links, 4 joints
Joints:
- joint rotor_joint: limit effort=500 velocity=5 -> effort=5000 velocity=50

Commit message: JTC action server added for better calibration

File: src/ros_deep_sampler/urdf/sampler_model.urdf (robot description, URDF)
Before this commit: robot slider_robot, 5 links, 4 joints
Joints:
- joint platform_joint: limit lower=-0.5 upper=0.5 effort=5000 velocity=0.5 -> lower=-0.5 upper=0.5 effort=5000 velocity=5.0

Commit message: added container joint

File: src/ros_deep_sampler/urdf/sampler_model.urdf (robot description, URDF)
Before this commit: robot slider_robot, 5 links, 4 joints
Links:
- added link container_link, mass 1.0; collision box size=0.7 0.1 0.02; visual box size=0.7 0.1 0.02
Joints:
- added joint container_joint: type revolute, parent base_link, child container_link, origin xyz=-0.2 0 -0.6 rpy=0 0 1.57, axis 0 0 1, limit lower=-1.6 upper=1.6 effort=20 velocity=2.0

Commit message: surface sample module in urdf + logic of new states

File: src/ros_deep_sampler/urdf/sampler_model.urdf (robot description, URDF)
Before this commit: robot slider_robot, 6 links, 5 joints
Links:
- added link brush_rotor_link, mass 0.5; collision box size=0.07 0.07 0.02; visual box size=0.07 0.07 0.02
- added link vaccum_body_link, mass 5; collision box size=0.4 0.3 0.5; visual box size=0.1 0.1 0.15
- added link vacuum_rotor_link, mass 0.5; collision box size=0.07 0.07 0.02; visual box size=0.07 0.07 0.02
- link container_link: geometry collision box size=0.7 0.1 0.02; visual box size=0.7 0.2 0.02
Joints:
- added joint brush_rotor_joint: type continuous, parent vaccum_body_link, child brush_rotor_link, origin xyz=0 0 -0.075 rpy=0 0 0, axis 0 0 1, limit effort=5000 velocity=50
- added joint vaccum_fixed_joint: type fixed, parent platform_link, child vaccum_body_link, origin xyz=0.2 0 -0.25 rpy=0 0 0
- added joint vacuum_rotor_joint: type continuous, parent vaccum_body_link, child vacuum_rotor_link, origin xyz=0 0 0.075 rpy=0 0 0, axis 0 0 1, limit effort=5000 velocity=50

Commit message: added clamp joint

File: src/ros_deep_sampler/urdf/sampler_model.urdf (robot description, URDF)
Before this commit: robot slider_robot, 9 links, 8 joints
Links:
- added link clamp_link, mass 0.5; collision box size=0.07 0.07 0.02; visual box size=0.07 0.07 0.02
- link vaccum_body_link: geometry collision box size=0.1 0.1 0.15; visual box size=0.1 0.1 0.15
Joints:
- added joint clamp_joint: type revolute, parent vaccum_body_link, child clamp_link, origin xyz=0.0 0.1 0.1 rpy=0 0 0, axis 1 0 0, limit lower=-1.6 upper=1.6 effort=100 velocity=20.0
- joint container_joint: limit lower=-1.6 upper=1.6 effort=20 velocity=2.0 -> lower=-1.6 upper=1.6 effort=100 velocity=10.0

Commit message: manual control via SET_RPM

File: src/ros_deep_sampler/urdf/sampler_model.urdf (robot description, URDF)
Before this commit: robot slider_robot, 10 links, 9 joints
Links:
- added link container_link1, mass 1.0; collision box size=0.7 0.1 0.02; visual box size=0.7 0.2 0.02
- added link drill_link1, mass 3.0; collision box size=0.05 0.6 0.05; visual box size=0.05 0.6 0.05
- added link platform_link1, mass 5.0; collision box size=0.1 0.6 0.1; visual box size=0.1 0.6 0.1
Joints:
- added joint container_vel_joint: type prismatic, parent base_link, child container_link1, origin xyz=0 0 5 rpy=0 0 1.57, axis 0 0 1, limit lower=-1.6 upper=1.6 effort=1000 velocity=5.0
- added joint drill_vel_joint: type prismatic, parent platform_link1, child drill_link1, origin xyz=0 0 0 rpy=0 0 0, axis 0 0 1, limit lower=-0.5 upper=0.5 effort=5000 velocity=5.0
- added joint platform_vel_joint: type prismatic, parent base_link, child platform_link1, origin xyz=0 0 5 rpy=0 0 0, axis 0 0 1, limit lower=-0.5 upper=0.5 effort=5000 velocity=5.0

Commit message: a small fix of manual control

File: src/ros_deep_sampler/urdf/sampler_model.urdf (robot description, URDF)
Before this commit: robot slider_robot, 13 links, 12 joints
Joints:
- joint container_joint: limit lower=-1.6 upper=1.6 effort=100 velocity=10.0 -> lower=-1.6 upper=1.6 effort=1000 velocity=10.0
